File: AmpliClase D.sch (KiCad schematic (older format))
At the start: 33 parts, among them Q1 IRF540N, Q2 IRF540N, Q3 MJE350, Q4 MJE340, Q5 MJE340, U1 TL494

Commit message: se cambian diodos
Parts:
- added D? (x2): D_Zener_ALT, symbol Device:D_Zener_ALT
- D2: value D_ALT -> 1n4148
Connections:
- net GND: now also D?.2 (A)
- net H_Side_Mosfet: now also D?.1 (K)
- net L_Node: now also D?.2 (A)
- net L_Side_Mosfet: now also D?.1 (K)
Other:
- note added: "12VDC"
Changed lines of the file:
@@
 P 4000 3800
 F 0 "D2" H 4000 3583 50  0000 C CNN
-F 1 "D_ALT" H 4000 3674 50  0000 C CNN
+F 1 "1n4148" H 4000 3674 50  0000 C CNN
 F 2 "" H 4000 3800 50  0001 C CNN
 F 3 "~" H 4000 3800 50  0001 C CNN
@@
 L_Side_Mosfet
 Wire Wire Line
-	3100 7950 3300 7950
-Wire Wire Line
-	3100 8800 3300 8800
+	3100 7950 3250 7950
 Wire Wire Line
 	3600 8600 3600 8350
 Wire Wire Line
-	3600 8350 3100 8350
+	3600 8350 3250 8350
 Connection ~ 3600 8350
 Wire Wire Line
@@
 $EndComp
 Wire Wire Line
-	3600 9300 3600 9000
+	3600 9300 3600 9200
 $Comp
 L power:VPP #PWR0111
@@
 Text Notes 3150 1800 0    50   ~ 0
 Audio + 2,5 V
+$Comp
+L Device:D_Zener_ALT D?
+U 1 1 61690AFA
+P 3250 8150
+F 0 "D?" V 3204 8229 50  0000 L CNN
+F 1 "D_Zener_ALT" V 3200 7550 50  0000 L CNN
+F 2 "" H 3250 8150 50  0001 C CNN
+F 3 "~" H 3250 8150 50  0001 C CNN
+	1    3250 8150
+	0    1    1    0
+$EndComp
+Wire Wire Line
+	3100 8800 3250 8800
+$Comp
+L Device:D_Zener_ALT D?
+U 1 1 61692510
+P 3250 9000
+F 0 "D?" V 3204 9079 50  0000 L CNN
+F 1 "D_Zener_ALT" V 3200 8400 50  0000 L CNN
+F 2 "" H 3250 9000 50  0001 C CNN
+F 3 "~" H 3250 9000 50  0001 C CNN
+	1    3250 9000
+	0    1    1    0
+$EndComp
+Wire Wire Line
+	3250 8000 3250 7950
+Connection ~ 3250 7950
+Wire Wire Line
+	3250 7950 3300 7950
+Wire Wire Line
+	3250 8300 3250 8350
+Connection ~ 3250 8350
+Wire Wire Line
+	3250 8350 3100 8350
+Wire Wire Line
+	3250 8850 3250 8800
+Connection ~ 3250 8800
+Wire Wire Line
+	3250 8800 3300 8800
+Wire Wire Line
+	3250 9150 3250 9200
+Wire Wire Line
+	3250 9200 3600 9200
+Connection ~ 3600 9200
+Wire Wire Line
+	3600 9200 3600 9000
+Text Notes 4750 900  0    50   ~ 0
+12VDC
 $EndSCHEMATC

Commit message: Changes to be committed: 	modified:   AmpliClase D-cache.lib 	modified:   AmpliClase D.net 	modified:   AmpliClase D.sch 	modified:   AmpliClase D.sch-bak 	new file:   Hojas de Datos/desktop.ini
Parts:
- D2: value 1n4148 -> D_ALT
- D5, D6: renamed from D?; value D_Zener_ALT -> 1n4739
Other:
- note added: "+12VDC"
- note removed: "12VDC"
Changed lines of the file:
@@
 EESchema Schematic File Version 4
-LIBS:AmpliClase D-cache
 EELAYER 30 0
 EELAYER END
@@
 P 4000 3800
 F 0 "D2" H 4000 3583 50  0000 C CNN
-F 1 "1n4148" H 4000 3674 50  0000 C CNN
+F 1 "D_ALT" H 4000 3674 50  0000 C CNN
 F 2 "" H 4000 3800 50  0001 C CNN
 F 3 "~" H 4000 3800 50  0001 C CNN
@@
 	4600 1200 4600 1550
 $Comp
-L power:VCC #PWR?
+L power:VCC #PWR0117
 U 1 1 6156A3CD
 P 5200 2050
-F 0 "#PWR?" H 5200 1900 50  0001 C CNN
+F 0 "#PWR0117" H 5200 1900 50  0001 C CNN
 F 1 "VCC" H 5215 2223 50  0000 C CNN
 F 2 "" H 5200 2050 50  0001 C CNN
@@
 Audio + 2,5 V
 $Comp
-L Device:D_Zener_ALT D?
+L Device:D_Zener_ALT D5
 U 1 1 61690AFA
 P 3250 8150
-F 0 "D?" V 3204 8229 50  0000 L CNN
-F 1 "D_Zener_ALT" V 3200 7550 50  0000 L CNN
+F 0 "D5" V 3204 8229 50  0000 L CNN
+F 1 "1n4739" V 3200 7550 50  0000 L CNN
 F 2 "" H 3250 8150 50  0001 C CNN
 F 3 "~" H 3250 8150 50  0001 C CNN
@@
 	3100 8800 3250 8800
 $Comp
-L Device:D_Zener_ALT D?
+L Device:D_Zener_ALT D6
 U 1 1 61692510
 P 3250 9000
-F 0 "D?" V 3204 9079 50  0000 L CNN
-F 1 "D_Zener_ALT" V 3200 8400 50  0000 L CNN
+F 0 "D6" V 3204 9079 50  0000 L CNN
+F 1 "1n4739" V 3200 8400 50  0000 L CNN
 F 2 "" H 3250 9000 50  0001 C CNN
 F 3 "~" H 3250 9000 50  0001 C CNN
@@
 	3600 9200 3600 9000
 Text Notes 4750 900  0    50   ~ 0
-12VDC
++12VDC
 $EndSCHEMATC

Commit message: modified:   AmpliClase D.sch 	modified:   AmpliClase D.sch-bak
Parts:
- D5, D6: value 1n4739 -> 1n4744A
Other:
- note added: "Diodos Zener de 15V"
Changed lines of the file:
@@
 P 3250 8150
 F 0 "D5" V 3204 8229 50  0000 L CNN
-F 1 "1n4739" V 3200 7550 50  0000 L CNN
+F 1 "1n4744A" V 3200 7550 50  0000 L CNN
 F 2 "" H 3250 8150 50  0001 C CNN
 F 3 "~" H 3250 8150 50  0001 C CNN
@@
 P 3250 9000
 F 0 "D6" V 3204 9079 50  0000 L CNN
-F 1 "1n4739" V 3200 8400 50  0000 L CNN
+F 1 "1n4744A" V 3200 8400 50  0000 L CNN
 F 2 "" H 3250 9000 50  0001 C CNN
 F 3 "~" H 3250 9000 50  0001 C CNN
@@
 Text Notes 4750 900  0    50   ~ 0
 +12VDC
+Text Notes 2500 8550 0    50   ~ 0
+Diodos Zener de 15V
 $EndSCHEMATC
